File: hardware/aa-daughterboard-lvds/aa-daughterboard-lvds.sch (KiCad schematic (older format))
At the start: 162 parts, among them CN1 Barrel_Jack, CN10 6P6C, CN11 6P6C, CN12 6P6C, CN13 6P6C, CN14 Conn_01x08, CN15 Conn_01x08, CN16 Conn_01x08, CN17 8P8C, CN18 8P8C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

Commit message: Second rount almost ready, less fiducials
Parts:
- D10, D11, D12, D13, D14, D15, D16, D17, D18, D19: value D5V0P4UR6SO -> DT1042
- F2, F3, F4, F5: footprint Fuse:Fuse_0603_1608Metric -> Fuse:Fuse_0805_2012Metric
- U3: footprint Package_TO_SOT_THT:TO-220-3_Vertical -> Package_TO_SOT_THT:TO-220-3_Horizontal_TabDown
Changed lines of the file:
@@
 EESchema Schematic File Version 4
-LIBS:aa-daughterboard-lvds-cache
 EELAYER 26 0
 EELAYER END
@@
 F 0 "U3" H 6850 1942 50  0000 C CNN
 F 1 "uA7805" H 6850 1851 50  0000 C CNN
-F 2 "Package_TO_SOT_THT:TO-220-3_Vertical" H 6875 1550 50  0001 L CIN
+F 2 "Package_TO_SOT_THT:TO-220-3_Horizontal_TabDown" H 6875 1550 50  0001 L CIN
 F 3 "" H 6850 1650 50  0001 C CNN
 	1    6850 1700
@@
 P 10050 10400
 F 0 "D12" H 10075 10865 50  0000 C CNN
-F 1 "D5V0P4UR6SO" H 10075 10774 50  0000 C CNN
+F 1 "DT1042" H 10075 10774 50  0000 C CNN
 F 2 "Package_TO_SOT_SMD:SOT-23-6" H 9500 10000 50  0001 L CNN
 F 3 "" V 10175 10275 50  0001 C CNN
@@
 P 10050 11700
 F 0 "D13" H 10075 12165 50  0000 C CNN
-F 1 "D5V0P4UR6SO" H 10075 12074 50  0000 C CNN
+F 1 "DT1042" H 10075 12074 50  0000 C CNN
 F 2 "Package_TO_SOT_SMD:SOT-23-6" H 9500 11300 50  0001 L CNN
 F 3 "" V 10175 11575 50  0001 C CNN
@@
 P 10050 6250
 F 0 "D10" H 10075 6715 50  0000 C CNN
-F 1 "D5V0P4UR6SO" H 10075 6624 50  0000 C CNN
+F 1 "DT1042" H 10075 6624 50  0000 C CNN
 F 2 "Package_TO_SOT_SMD:SOT-23-6" H 9500 5850 50  0001 L CNN
 F 3 "" V 10175 6125 50  0001 C CNN
@@
 P 10050 7550
 F 0 "D11" H 10075 8015 50  0000 C CNN
-F 1 "D5V0P4UR6SO" H 10075 7924 50  0000 C CNN
+F 1 "DT1042" H 10075 7924 50  0000 C CNN
 F 2 "Package_TO_SOT_SMD:SOT-23-6" H 9500 7150 50  0001 L CNN
 F 3 "" V 10175 7425 50  0001 C CNN
@@
 P 18350 3650
 F 0 "D14" H 18375 4115 50  0000 C CNN
-F 1 "D5V0P4UR6SO" H 18375 4024 50  0000 C CNN
+F 1 "DT1042" H 18375 4024 50  0000 C CNN
 F 2 "Package_TO_SOT_SMD:SOT-23-6" H 17800 3250 50  0001 L CNN
 F 3 "" V 18475 3525 50  0001 C CNN
@@
 P 18350 4950
 F 0 "D15" H 18375 5415 50  0000 C CNN
-F 1 "D5V0P4UR6SO" H 18375 5324 50  0000 C CNN
+F 1 "DT1042" H 18375 5324 50  0000 C CNN
 F 2 "Package_TO_SOT_SMD:SOT-23-6" H 17800 4550 50  0001 L CNN
 F 3 "" V 18475 4825 50  0001 C CNN
@@
 P 18350 11750
 F 0 "D18" H 18375 12215 50  0000 C CNN
-F 1 "D5V0P4UR6SO" H 18375 12124 50  0000 C CNN
+F 1 "DT1042" H 18375 12124 50  0000 C CNN
 F 2 "Package_TO_SOT_SMD:SOT-23-6" H 17800 11350 50  0001 L CNN
 F 3 "" V 18475 11625 50  0001 C CNN
@@
 P 18350 13050
 F 0 "D19" H 18375 13515 50  0000 C CNN
-F 1 "D5V0P4UR6SO" H 18375 13424 50  0000 C CNN
+F 1 "DT1042" H 18375 13424 50  0000 C CNN
 F 2 "Package_TO_SOT_SMD:SOT-23-6" H 17800 12650 50  0001 L CNN
 F 3 "" V 18475 12925 50  0001 C CNN
@@
 P 18350 7750
 F 0 "D16" H 18375 8215 50  0000 C CNN
-F 1 "D5V0P4UR6SO" H 18375 8124 50  0000 C CNN
+F 1 "DT1042" H 18375 8124 50  0000 C CNN
 F 2 "Package_TO_SOT_SMD:SOT-23-6" H 17800 7350 50  0001 L CNN
 F 3 "" V 18475 7625 50  0001 C CNN
@@
 P 18350 9050
 F 0 "D17" H 18375 9515 50  0000 C CNN
-F 1 "D5V0P4UR6SO" H 18375 9424 50  0000 C CNN
+F 1 "DT1042" H 18375 9424 50  0000 C CNN
 F 2 "Package_TO_SOT_SMD:SOT-23-6" H 17800 8650 50  0001 L CNN
 F 3 "" V 18475 8925 50  0001 C CNN
@@
 F 0 "F2" V 11475 5650 50  0000 C CNN
 F 1 "0.5A" V 11566 5650 50  0000 C CNN
-F 2 "Fuse:Fuse_0603_1608Metric" H 11750 5450 50  0001 L CNN
+F 2 "Fuse:Fuse_0805_2012Metric" H 11750 5450 50  0001 L CNN
 F 3 "~" H 11700 5650 50  0001 C CNN
 	1    11700 5650
@@
 F 0 "F3" V 11475 7400 50  0000 C CNN
 F 1 "0.5A" V 11566 7400 50  0000 C CNN
-F 2 "Fuse:Fuse_0603_1608Metric" H 11750 7200 50  0001 L CNN
+F 2 "Fuse:Fuse_0805_2012Metric" H 11750 7200 50  0001 L CNN
 F 3 "~" H 11700 7400 50  0001 C CNN
 	1    11700 7400
@@
 F 0 "F4" V 11475 9800 50  0000 C CNN
 F 1 "0.5A" V 11566 9800 50  0000 C CNN
-F 2 "Fuse:Fuse_0603_1608Metric" H 11750 9600 50  0001 L CNN
+F 2 "Fuse:Fuse_0805_2012Metric" H 11750 9600 50  0001 L CNN
 F 3 "~" H 11700 9800 50  0001 C CNN
 	1    11700 9800
@@
 F 0 "F5" V 11475 11550 50  0000 C CNN
 F 1 "0.5A" V 11566 11550 50  0000 C CNN
-F 2 "Fuse:Fuse_0603_1608Metric" H 11750 11350 50  0001 L CNN
+F 2 "Fuse:Fuse_0805_2012Metric" H 11750 11350 50  0001 L CNN
 F 3 "~" H 11700 11550 50  0001 C CNN
 	1    11700 11550
