File: hardware/aa-daughterboard-lvds/aa-daughterboard-lvds.kicad_pcb (KiCad board)
At the start: 4 copper layers, 175.3 x 96.5 mm, 167 parts, among them CN1 Barrel_Jack, CN10 6P6C, CN11 6P6C, CN12 6P6C, CN13 6P6C, CN14 Conn_01x08, CN15 Conn_01x08, CN16 Conn_01x08, CN17 8P8C, CN18 8P8C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

Commit message: Fix silkscreen for stalk connectors
Other:
- board text removed: "PN"
Changed lines of the file:
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@@
     (34 B.Paste user)
     (35 F.Paste user)
-    (36 B.SilkS user hide)
-    (37 F.SilkS user hide)
+    (36 B.SilkS user)
+    (37 F.SilkS user)
     (38 B.Mask user hide)
     (39 F.Mask user hide)
@@
     (effects (font (size 0.762 0.762) (thickness 0.1016)) (justify mirror))
   )
-  (gr_text PN (at 204.216 63.5 90) (layer B.SilkS)
+  (gr_text CN (at 204.216 63.5 90) (layer B.SilkS)
     (effects (font (size 0.762 0.762) (thickness 0.1016)) (justify mirror))
   )
