File: hardware/aa-panel-receiver-lvds/aa-panel-receiver-lvds.sch (KiCad schematic (older format))
At the start: 30 parts, among them CN10 6P6C, CN11 6P6C, CN2 Conn_01x02, CN6 Conn_01x04, CN7 Conn_01x04, U4 75ALS192

Commit message: More updates to daughterboard, begin panel receiver layout
Parts:
- removed CN11: 6P6C, aa-panel-receiver-lvds:6P6C_Assmann_A-2014-1-4, symbol Connector:6P6C
- removed CN7: Conn_01x04, Connector_PinHeader_2.54mm:PinHeader_1x04_P2.54mm_Vertical, symbol Connector_Generic:Conn_01x04
- removed D11: D5V0P4UR6SO, Package_TO_SOT_SMD:SOT-23-6, symbol aa-panel-receiver-lvds:D5V0P4UR6SO
- removed D3: DF2S16FS, aa-panel-receiver-lvds:D_SOD-923, symbol Device:D_Zener
- removed F1: 500mA, aa-panel-receiver-lvds:Fuseholder_Clip_5x20_Bel_FC-211-22, symbol Device:Fuse
- removed R16, R17, R18, R19, R24, R25, R26, R27: 56, Resistor_SMD:R_0603_1608Metric, symbol Device:R
- removed TP21, TP22, TP31: TestPoint, TestPoint:TestPoint_THTPad_D1.0mm_Drill0.5mm, symbol Connector:TestPoint
- removed U4: 75ALS192, Package_SO:SOIC-16_3.9x9.9mm_P1.27mm, symbol aa-panel-receiver-lvds:75ALS192
- added C2: 1u, Capacitor_SMD:C_0805_2012Metric, symbol Device:C
- added C3, C4, C7: 0.1u, Capacitor_SMD:C_0805_2012Metric, symbol Device:C
- added C8: 100u, Capacitor_THT:CP_Radial_D10.0mm_P2.50mm_P5.00mm, symbol Device:CP
- added C9: 10u, Capacitor_SMD:C_0805_2012Metric, symbol Device:C
- added D2: D5V0P4UR6SO, Package_TO_SOT_SMD:SOT-23-6, symbol aa-panel-receiver-lvds:D5V0P4UR6SO
- added J1: Conn_01x08, Connector_PinHeader_2.54mm:PinHeader_1x04_P2.54mm_Vertical, symbol Connector_Generic:Conn_01x04
- added R1, R2, R3, R4, R5, R6, R7, R8: 56, Resistor_SMD:R_0603_1608Metric, symbol Device:R
- added R10, R9: 10k, Resistor_SMD:R_0603_1608Metric, symbol Device:R
- added TP1, TP11, TP2, TP4, TP5, TP6, TP7, TP8, TP9: TestPoint, TestPoint:TestPoint_THTPad_D2.0mm_Drill1.0mm, symbol Connector:TestPoint
- added U1: MC3486N, Package_SO:SOIC-16_3.9x9.9mm_P1.27mm, symbol Interface_LineDriver:MC3486N
- added U2: Si8640EB-B-IU, Package_SO:QSOP-16_3.9x4.9mm_P0.635mm, symbol Isolator:Si8640EB-B-IU
- added U3: LM4562, Package_SO:SOIC-8_3.9x4.9mm_P1.27mm, symbol Amplifier_Operational:LM4562
- added U4: CRE1S0505S3C, Converter_DCDC:Converter_DCDC_muRata_CRE1xxxxxx3C_THT, symbol Regulator_Switching:CRE1S0505S3C
- C5: value 10u -> 0.1u
- C6: footprint Capacitor_SMD:C_0603_1608Metric -> Capacitor_SMD:C_0805_2012Metric
- CN1: renamed from CN6; footprint Connector_PinHeader_2.54mm:PinHeader_1x04_P2.54mm_Vertical -> Connector_PinHeader_2.54mm:PinHeader_2x04_P2.54mm_Vertical; symbol Connector_Generic:Conn_01x04 -> Connector_Generic:Conn_01x08
- CN2: renamed from CN10; value 6P6C -> 8P8C; footprint aa-panel-receiver-lvds:6P6C_Assmann_A-2014-1-4 -> aa-panel-receiver-lvds:8P8C_Assmann_A-2014-2S-4; symbol Connector:6P6C -> Connector:8P8C_Shielded
- CN3: renamed from CN2; footprint Connector_Wire:SolderWirePad_1x02_P7.62mm_Drill2.5mm -> Connector_Wire:SolderWirePad_1x02_P5.08mm_Drill1.5mm
- TP10: renamed from TP30; footprint TestPoint:TestPoint_THTPad_D1.0mm_Drill0.5mm -> TestPoint:TestPoint_THTPad_D2.0mm_Drill1.0mm
- TP3: footprint TestPoint:TestPoint_THTPad_D1.0mm_Drill0.5mm -> TestPoint:TestPoint_THTPad_D2.0mm_Drill1.0mm
- renumbered C8 to C1, D10 to D1
Connections:
- net labels added: +2.5A, +2.5B, +5V_SX, +5V_X, GND_S, GND_XY, IN_TX_PANEL_0_N, IN_TX_PANEL_0_P, IN_TX_PANEL_1_N, IN_TX_PANEL_1_P, IN_TX_PANEL_2_N, IN_TX_PANEL_2_P, IN_TX_PANEL_3_N, IN_TX_PANEL_3_P
- net labels removed: +5V, PWM_CAP_1, PWM_CAP_1_N, PWM_CAP_1_P, PWM_CAP_B, PWM_CAP_B_N, PWM_CAP_B_P, TX_STALK_1, TX_STALK_1_N, TX_STALK_1_P, TX_STALK_B, TX_STALK_B_N, TX_STALK_B_P
- wire segments 143 -> 264
Other:
- moved on the sheet: C1, CN3, H1, H2, H3, H4, TP10

Commit message: Add power distro board, resolve some todos, finish a coherent layout of the panel receiver
Parts:
- removed C2: 1u, Capacitor_SMD:C_0805_2012Metric, symbol Device:C
- added D3, D4: LED, Diode_SMD:D_0603_1608Metric, symbol Device:LED
- added R11, R12: 470, Resistor_SMD:R_0603_1608Metric, symbol Device:R
- CN4: renamed from J1; footprint Connector_PinHeader_2.54mm:PinHeader_1x04_P2.54mm_Vertical -> Connector_PinHeader_2.54mm:PinHeader_2x04_P2.54mm_Vertical; symbol Connector_Generic:Conn_01x04 -> Connector_Generic:Conn_01x08
Connections:
- net labels added: +5V_S, IN_TX_PANEL_0, IN_TX_PANEL_1, IN_TX_PANEL_2, IN_TX_PANEL_3, TX_PANEL_0, TX_PANEL_1, TX_PANEL_2, TX_PANEL_3
- net labels removed: +5V_SX, GND_XY
- wire segments 264 -> 289
Other:
- moved on the sheet: C1, C3, C5, CN1, CN2, CN3, TP1, TP10, TP11, TP2

Commit message: Update to use a shared schematic component/footprint library
Parts:
- CN2: footprint aa-panel-receiver-lvds:8P8C_Assmann_A-2014-2S-4 -> aa-shared:8P8C_Assmann_A-2014-2S-4
- D1, D2: symbol aa-panel-receiver-lvds:D5V0P4UR6SO -> aa-shared:D5V0P4UR6SO
Changed lines of the file:
@@
 $EndComp
 $Comp
-L aa-panel-receiver-lvds:D5V0P4UR6SO D1
+L aa-shared:D5V0P4UR6SO D1
 U 1 1 5FA1B995
 P 7850 5700
@@
 	14200 5950 14200 5500
 $Comp
-L aa-panel-receiver-lvds:+5V_X #PWR033
+L aa-shared:+5V_X #PWR033
 U 1 1 5D2F4E2D
 P 15350 10200
@@
 	8900 2300 9150 2300
 $Comp
-L aa-panel-receiver-lvds:+5V_X #PWR019
+L aa-shared:+5V_X #PWR019
 U 1 1 5D3F39C5
 P 14200 5450
@@
 	14400 5850 14400 5900
 $Comp
-L aa-panel-receiver-lvds:+5V_S #PWR011
+L aa-shared:+5V_S #PWR011
 U 1 1 5EA9F454
 P 11300 7600
@@
 $EndComp
 $Comp
-L aa-panel-receiver-lvds:+5V_S #PWR015
+L aa-shared:+5V_S #PWR015
 U 1 1 5EA9F5A2
 P 11600 7150
@@
 $EndComp
 $Comp
-L aa-panel-receiver-lvds:+5V_S #PWR014
+L aa-shared:+5V_S #PWR014
 U 1 1 5EAA0590
 P 11600 4950
@@
 $EndComp
 $Comp
-L aa-panel-receiver-lvds:+5V_S #PWR05
+L aa-shared:+5V_S #PWR05
 U 1 1 5EAA0637
 P 11300 3700
@@
 $EndComp
 $Comp
-L aa-panel-receiver-lvds:+5V_S #PWR017
+L aa-shared:+5V_S #PWR017
 U 1 1 5EAA06DE
 P 13200 5500
@@
 $EndComp
 $Comp
-L aa-panel-receiver-lvds:+5V_S #PWR025
+L aa-shared:+5V_S #PWR025
 U 1 1 5EAA57F8
 P 8900 9850
@@
 $EndComp
 $Comp
-L aa-panel-receiver-lvds:+5V_S #PWR027
+L aa-shared:+5V_S #PWR027
 U 1 1 5EAA651D
 P 9850 9600
@@
 $EndComp
 $Comp
-L aa-panel-receiver-lvds:+5V_S #PWR029
+L aa-shared:+5V_S #PWR029
 U 1 1 5EAA6FD2
 P 11350 10150
@@
 $EndComp
 $Comp
-L aa-panel-receiver-lvds:GND_S #PWR012
+L aa-shared:GND_S #PWR012
 U 1 1 5EAB4727
 P 11300 8250
@@
 $EndComp
 $Comp
-L aa-panel-receiver-lvds:GND_S #PWR04
+L aa-shared:GND_S #PWR04
 U 1 1 5EAB47CE
 P 8250 7450
@@
 $EndComp
 $Comp
-L aa-panel-receiver-lvds:GND_S #PWR010
+L aa-shared:GND_S #PWR010
 U 1 1 5EAB4875
 P 11300 7150
@@
 $EndComp
 $Comp
-L aa-panel-receiver-lvds:GND_S #PWR06
+L aa-shared:GND_S #PWR06
 U 1 1 5EAB5562
 P 11300 4950
@@
 $EndComp
 $Comp
-L aa-panel-receiver-lvds:GND_S #PWR013
+L aa-shared:GND_S #PWR013
 U 1 1 5EAB5609
 P 11550 4150
@@
 $EndComp
 $Comp
-L aa-panel-receiver-lvds:GND_S #PWR018
+L aa-shared:GND_S #PWR018
 U 1 1 5EAB668A
 P 13200 6850
@@
 $EndComp
 $Comp
-L aa-panel-receiver-lvds:GND_S #PWR016
+L aa-shared:GND_S #PWR016
 U 1 1 5EAB6731
 P 13000 6000
@@
 F 0 "CN2" H 4370 6204 50  0000 R CNN
 F 1 "8P8C" H 4370 6295 50  0000 R CNN
-F 2 "aa-panel-receiver-lvds:8P8C_Assmann_A-2014-2S-4" V 4700 6225 50  0001 C CNN
+F 2 "aa-shared:8P8C_Assmann_A-2014-2S-4" V 4700 6225 50  0001 C CNN
 F 3 "~" V 4700 6225 50  0001 C CNN
 	1    4700 6200
@@
 $EndComp
 $Comp
-L aa-panel-receiver-lvds:GND_S #PWR02
+L aa-shared:GND_S #PWR02
 U 1 1 5EAB83F8
 P 5150 3100
@@
 $EndComp
 $Comp
-L aa-panel-receiver-lvds:GND_S #PWR01
+L aa-shared:GND_S #PWR01
 U 1 1 5EAB849F
 P 4950 5550
@@
 $EndComp
 $Comp
-L aa-panel-receiver-lvds:GND_S #PWR022
+L aa-shared:GND_S #PWR022
 U 1 1 5EAB8546
 P 7350 11200
@@
 $EndComp
 $Comp
-L aa-panel-receiver-lvds:GND_S #PWR023
+L aa-shared:GND_S #PWR023
 U 1 1 5EABA649
 P 8100 10600
@@
 $EndComp
 $Comp
-L aa-panel-receiver-lvds:GND_S #PWR024
+L aa-shared:GND_S #PWR024
 U 1 1 5EABA6F0
 P 8100 11800
@@
 $EndComp
 $Comp
-L aa-panel-receiver-lvds:GND_S #PWR026
+L aa-shared:GND_S #PWR026
 U 1 1 5EABAAC8
 P 8900 10550
@@
 $EndComp
 $Comp
-L aa-panel-receiver-lvds:GND_S #PWR028
+L aa-shared:GND_S #PWR028
 U 1 1 5EABAB6F
 P 9850 10600
@@
 $EndComp
 $Comp
-L aa-panel-receiver-lvds:GND_S #PWR030
+L aa-shared:GND_S #PWR030
 U 1 1 5EABC7F8
 P 12250 10750
@@
 $EndComp
 $Comp
-L aa-panel-receiver-lvds:GND_S #PWR031
+L aa-shared:GND_S #PWR031
 U 1 1 5EB9A533
 P 8900 2400
@@
 	13000 10250 13250 10250
 $Comp
-L aa-panel-receiver-lvds:+5V_S #PWR0101
+L aa-shared:+5V_S #PWR0101
 U 1 1 5F3CF015
 P 8250 5050
@@
 	11300 6500 11300 6550
 $Comp
-L aa-panel-receiver-lvds:+5V_S #PWR09
+L aa-shared:+5V_S #PWR09
 U 1 1 5EA9F4FB
 P 11300 6500
@@
 $EndComp
 $Comp
-L aa-panel-receiver-lvds:GND_S #PWR08
+L aa-shared:GND_S #PWR08
 U 1 1 5EAB54BB
 P 11300 6050
@@
 $EndComp
 $Comp
-L aa-panel-receiver-lvds:+5V_S #PWR07
+L aa-shared:+5V_S #PWR07
 U 1 1 5EAA04E9
 P 11300 5400
@@
 	11600 6100 11600 6050
 $Comp
-L aa-panel-receiver-lvds:+5V_S #PWR0103
+L aa-shared:+5V_S #PWR0103
 U 1 1 5F431B34
 P 11600 6050
@@
 	11600 8300 11600 8250
 $Comp
-L aa-panel-receiver-lvds:+5V_S #PWR0104
+L aa-shared:+5V_S #PWR0104
 U 1 1 5F431BD7
 P 11600 8250
@@
 	7250 7000 7550 7000
 $Comp
-L aa-panel-receiver-lvds:D5V0P4UR6SO D2
+L aa-shared:D5V0P4UR6SO D2
 U 1 1 5D094592
 P 7900 7150
@@
 $EndComp
 $Comp
-L aa-panel-receiver-lvds:GND_S #PWR03
+L aa-shared:GND_S #PWR03
 U 1 1 64DBE017
 P 11900 11000

Commit message: Substantial rework of system, new layouts done for daughterboard, power, stalk receiver
Parts:
- removed R10, R9: 10k, Resistor_SMD:R_0603_1608Metric, symbol Device:R
- removed TP3, TP4, TP7: TestPoint, TestPoint:TestPoint_THTPad_D2.0mm_Drill1.0mm, symbol Connector:TestPoint
- removed U3: LM4562, Package_SO:SOIC-8_3.9x4.9mm_P1.27mm, symbol Amplifier_Operational:LM4562
- added C301: 1u, Capacitor_SMD:C_0603_1608Metric, symbol Device:C
- added C302, C303, C304, C311, C321: 0.1u, Capacitor_SMD:C_0603_1608Metric, symbol Device:C
- added CN101: Conn_01x02, Connector_Wire:SolderWirePad_1x02_P5.08mm_Drill1.5mm, symbol Connector_Generic:Conn_01x02
- added CN301: 8P8C, aa-shared:8P8C_Assmann_A-2014-2S-4, symbol Connector:8P8C_Shielded
- added CN302: Conn_01x08, Connector_PinHeader_2.54mm:PinHeader_2x04_P2.54mm_Vertical, symbol Connector_Generic:Conn_01x08
- added CN351: Conn_01x04, Connector_PinHeader_2.54mm:PinHeader_1x04_P2.54mm_Vertical, symbol Connector_Generic:Conn_01x08
- added D101, D102: TSS83L45, aa-shared:D_SOD-128, symbol Device:D_Schottky
- added D211, D212, D221, D222, D311, D312, D321, D322: D_Zener, Diode_THT:D_DO-35_SOD27_P2.54mm_Vertical_KathodeUp, symbol Device:D_Zener
- added D301, D302: D5V0P4UR6SO, Package_TO_SOT_SMD:SOT-23-6, symbol aa-shared:D5V0P4UR6SO
- added R301, R302, R303, R304, R305, R306, R307, R308: 56, Resistor_SMD:R_0603_1608Metric, symbol Device:R
- added TP102, TP152, TP261, TP311, TP321, TP351, TP352, TP353, TP354, TP361, TP371, TP?: TestPoint, aa-shared:TestPoint_Loop_D1.80mm_Drill1.0mm_Beaded, symbol Connector:TestPoint
- added TP201: D0, aa-shared:TestPoint_Loop_D1.80mm_Drill1.0mm_Beaded, symbol Connector:TestPoint
- added TP202: D1, aa-shared:TestPoint_Loop_D1.80mm_Drill1.0mm_Beaded, symbol Connector:TestPoint
- added TP203: D2, aa-shared:TestPoint_Loop_D1.80mm_Drill1.0mm_Beaded, symbol Connector:TestPoint
- added TP204: D3, aa-shared:TestPoint_Loop_D1.80mm_Drill1.0mm_Beaded, symbol Connector:TestPoint
- added TP253, TP254: GND, aa-shared:TestPoint_Loop_D1.80mm_Drill1.0mm_Beaded, symbol Connector:TestPoint
- added TP301: D4, aa-shared:TestPoint_Loop_D1.80mm_Drill1.0mm_Beaded, symbol Connector:TestPoint
- added TP302: D5, aa-shared:TestPoint_Loop_D1.80mm_Drill1.0mm_Beaded, symbol Connector:TestPoint
- added TP303: D6, aa-shared:TestPoint_Loop_D1.80mm_Drill1.0mm_Beaded, symbol Connector:TestPoint
- added TP304: D7, aa-shared:TestPoint_Loop_D1.80mm_Drill1.0mm_Beaded, symbol Connector:TestPoint
- added U301: ST26C32, Package_DIP:DIP-14_W7.62mm, symbol Interface_LineDriver:MC3486N
- added U302: Si8640EB-B-IU, Package_SO:QSOP-16_3.9x4.9mm_P0.635mm, symbol Isolator:Si8640EB-B-IU
- C102: renamed from C9; footprint Capacitor_SMD:C_0805_2012Metric -> Capacitor_THT:CP_Radial_D6.3mm_P2.50mm
- C201: renamed from C1; footprint Capacitor_SMD:C_0805_2012Metric -> Capacitor_SMD:C_0603_1608Metric
- C202: renamed from C3; footprint Capacitor_SMD:C_0805_2012Metric -> Capacitor_SMD:C_0603_1608Metric
- C203: renamed from C4; footprint Capacitor_SMD:C_0805_2012Metric -> Capacitor_SMD:C_0603_1608Metric
- C204: renamed from C5; footprint Capacitor_SMD:C_0805_2012Metric -> Capacitor_SMD:C_0603_1608Metric
- C211: renamed from C6; footprint Capacitor_SMD:C_0805_2012Metric -> Capacitor_SMD:C_0603_1608Metric
- C221: renamed from C7; footprint Capacitor_SMD:C_0805_2012Metric -> Capacitor_SMD:C_0603_1608Metric
- CN251: renamed from CN1; footprint Connector_PinHeader_2.54mm:PinHeader_2x04_P2.54mm_Vertical -> Connector_PinHeader_2.54mm:PinHeader_1x04_P2.54mm_Vertical
- D151: renamed from D3; footprint Diode_SMD:D_0603_1608Metric -> LED_SMD:LED_0603_1608Metric
- D152: renamed from D4; footprint Diode_SMD:D_0603_1608Metric -> LED_SMD:LED_0603_1608Metric
- H1, H2, H3, H4: footprint MountingHole:MountingHole_4.3mm_M4_Pad_Via -> MountingHole:MountingHole_2.7mm_M2.5_Pad_Via
- TP101: renamed from TP8; footprint TestPoint:TestPoint_THTPad_D2.0mm_Drill1.0mm -> aa-shared:TestPoint_Loop_D1.80mm_Drill1.0mm_Beaded
- TP103: renamed from TP10; footprint TestPoint:TestPoint_THTPad_D2.0mm_Drill1.0mm -> aa-shared:TestPoint_Loop_D1.80mm_Drill1.0mm_Beaded
- TP151: renamed from TP9; footprint TestPoint:TestPoint_THTPad_D2.0mm_Drill1.0mm -> aa-shared:TestPoint_Loop_D1.80mm_Drill1.0mm_Beaded
- TP153: renamed from TP11; footprint TestPoint:TestPoint_THTPad_D2.0mm_Drill1.0mm -> aa-shared:TestPoint_Loop_D1.80mm_Drill1.0mm_Beaded
- TP211: renamed from TP5; footprint TestPoint:TestPoint_THTPad_D2.0mm_Drill1.0mm -> aa-shared:TestPoint_Loop_D1.80mm_Drill1.0mm_Beaded
- TP221: renamed from TP6; footprint TestPoint:TestPoint_THTPad_D2.0mm_Drill1.0mm -> aa-shared:TestPoint_Loop_D1.80mm_Drill1.0mm_Beaded
- TP251: renamed from TP1; footprint TestPoint:TestPoint_THTPad_D2.0mm_Drill1.0mm -> aa-shared:TestPoint_Loop_D1.80mm_Drill1.0mm_Beaded
- TP252: renamed from TP2; footprint TestPoint:TestPoint_THTPad_D2.0mm_Drill1.0mm -> aa-shared:TestPoint_Loop_D1.80mm_Drill1.0mm_Beaded
- U201: renamed from U1; value MC3486N -> ST26C32; footprint Package_SO:SOIC-16_3.9x9.9mm_P1.27mm -> Package_DIP:DIP-14_W7.62mm
- renumbered C8 to C101, CN3 to CN102, CN2 to CN201, CN4 to CN202, D1 to D201, D2 to D202, R11 to R151, R12 to R152, R1 to R201, R2 to R202, R3 to R203, R4 to R204, R5 to R205, R6 to R206, R7 to R207, R8 to R208, U4 to U101, U2 to U202
Connections:
- net labels added: +5V, +5V_Y, PANEL_0, PANEL_0_N, PANEL_0_P, PANEL_0_S, PANEL_1, PANEL_1_N, PANEL_1_P, PANEL_1_S, PANEL_2, PANEL_2_N, PANEL_2_P, PANEL_2_S, PANEL_3, PANEL_3_N, PANEL_3_P, PANEL_3_S, PANEL_4, PANEL_4_N, PANEL_4_P, PANEL_4_S, PANEL_5, PANEL_5_N, PANEL_5_P, PANEL_5_S, PANEL_6, PANEL_6_N, PANEL_6_P, PANEL_6_S, PANEL_7, PANEL_7_N, PANEL_7_P, PANEL_7_S
- net labels removed: IN_TX_PANEL_0, IN_TX_PANEL_0_N, IN_TX_PANEL_0_P, IN_TX_PANEL_1, IN_TX_PANEL_1_N, IN_TX_PANEL_1_P, IN_TX_PANEL_2, IN_TX_PANEL_2_N, IN_TX_PANEL_2_P, IN_TX_PANEL_3, IN_TX_PANEL_3_N, IN_TX_PANEL_3_P, TX_PANEL_0, TX_PANEL_1, TX_PANEL_2, TX_PANEL_3
- wire segments 289 -> 555
Other:
- moved on the sheet: C101, C102, C201, C202, C203, C204, C211, C221, CN102, CN201, CN202, CN251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

Commit message: Renumber and duplicate layout for panel receiver -- layout not complete
Parts:
- CN251, CN351: value Conn_01x04 -> Conn_01x08; footprint Connector_PinHeader_2.54mm:PinHeader_1x04_P2.54mm_Vertical -> Connector_PinHeader_2.54mm:PinHeader_2x04_P2.54mm_Vertical
- U201, U301: footprint Package_DIP:DIP-14_W7.62mm -> Package_SO:SOIC-16_3.9x9.9mm_P1.27mm
- gave numbers to parts that had none: 1
Connections:
- net +5V_X: no longer C304.1, U302.10 (EN2), U302.16 (VDD2)
- net +5V_Y: now also C304.1, U302.10 (EN2), U302.16 (VDD2)
Changed lines of the file:
@@
 P 4150 3700
 F 0 "CN251" H 4229 3646 50  0000 L CNN
-F 1 "Conn_01x04" H 4230 3601 50  0001 L CNN
-F 2 "Connector_PinHeader_2.54mm:PinHeader_1x04_P2.54mm_Vertical" H 4150 3700 50  0001 C CNN
+F 1 "Conn_01x08" H 4230 3601 50  0001 L CNN
+F 2 "Connector_PinHeader_2.54mm:PinHeader_2x04_P2.54mm_Vertical" H 4150 3700 50  0001 C CNN
 F 3 "" H 4150 3700 50  0001 C CNN
 	1    4150 3700
@@
 Connection ~ 10350 4200
 Connection ~ 10350 5300
-$Comp
-L power:PWR_FLAG #FLG04
-U 1 1 5D3EBFCB
-P 12000 1950
-F 0 "#FLG04" H 12000 2025 50  0001 C CNN
-F 1 "PWR_FLAG" H 12000 2124 50  0001 C CNN
-F 2 "" H 12000 1950 50  0001 C CNN
-F 3 "" H 12000 1950 50  0001 C CNN
-	1    12000 1950
-	1    0    0    1
-$EndComp
 Wire Wire Line
 	10250 5300 10350 5300
@@
 F 0 "U201" H 12350 7450 50  0000 C CNN
 F 1 "ST26C32" H 12550 7600 50  0000 L CNN
-F 2 "Package_DIP:DIP-14_W7.62mm" H 12400 7050 50  0001 C CNN
+F 2 "Package_SO:SOIC-16_3.9x9.9mm_P1.27mm" H 12400 7050 50  0001 C CNN
 F 3 "" H 12400 7450 50  0001 C CNN
 	3    12400 7450
@@
 F 0 "U201" H 12350 4550 50  0000 C CNN
 F 1 "ST26C32" H 12500 4700 50  0000 L CNN
-F 2 "Package_DIP:DIP-14_W7.62mm" H 12400 4150 50  0001 C CNN
+F 2 "Package_SO:SOIC-16_3.9x9.9mm_P1.27mm" H 12400 4150 50  0001 C CNN
 F 3 "" H 12400 4550 50  0001 C CNN
 	1    12400 4550
@@
 F 0 "U201" H 12350 5650 50  0000 C CNN
 F 1 "ST26C32" H 12550 5800 50  0000 L CNN
-F 2 "Package_DIP:DIP-14_W7.62mm" H 12400 5250 50  0001 C CNN
+F 2 "Package_SO:SOIC-16_3.9x9.9mm_P1.27mm" H 12400 5250 50  0001 C CNN
 F 3 "" H 12400 5650 50  0001 C CNN
 	2    12400 5650
@@
 F 0 "U201" H 12350 8550 50  0000 C CNN
 F 1 "ST26C32" H 12550 8700 50  0000 L CNN
-F 2 "Package_DIP:DIP-14_W7.62mm" H 12400 8150 50  0001 C CNN
+F 2 "Package_SO:SOIC-16_3.9x9.9mm_P1.27mm" H 12400 8150 50  0001 C CNN
 F 3 "" H 12400 8550 50  0001 C CNN
 	4    12400 8550
@@
 Wire Wire Line
 	12150 1850 12200 1850
-Wire Wire Line
-	11850 1950 12000 1950
-Connection ~ 12000 1950
-Wire Wire Line
-	12000 1950 12150 1950
 $Comp
 L Connector:TestPoint TP153
@@
 P 4550 10250
 F 0 "CN351" H 4629 10196 50  0000 L CNN
-F 1 "Conn_01x04" H 4630 10151 50  0001 L CNN
-F 2 "Connector_PinHeader_2.54mm:PinHeader_1x04_P2.54mm_Vertical" H 4550 10250 50  0001 C CNN
+F 1 "Conn_01x08" H 4630 10151 50  0001 L CNN
+F 2 "Connector_PinHeader_2.54mm:PinHeader_2x04_P2.54mm_Vertical" H 4550 10250 50  0001 C CNN
 F 3 "" H 4550 10250 50  0001 C CNN
 	1    4550 10250
@@
 F 0 "U301" H 12750 14000 50  0000 C CNN
 F 1 "ST26C32" H 12950 14150 50  0000 L CNN
-F 2 "Package_DIP:DIP-14_W7.62mm" H 12800 13600 50  0001 C CNN
+F 2 "Package_SO:SOIC-16_3.9x9.9mm_P1.27mm" H 12800 13600 50  0001 C CNN
 F 3 "" H 12800 14000 50  0001 C CNN
 	3    12800 14000
@@
 F 0 "U301" H 12750 11100 50  0000 C CNN
 F 1 "ST26C32" H 12900 11250 50  0000 L CNN
-F 2 "Package_DIP:DIP-14_W7.62mm" H 12800 10700 50  0001 C CNN
+F 2 "Package_SO:SOIC-16_3.9x9.9mm_P1.27mm" H 12800 10700 50  0001 C CNN
 F 3 "" H 12800 11100 50  0001 C CNN
 	1    12800 11100
@@
 F 0 "U301" H 12750 12200 50  0000 C CNN
 F 1 "ST26C32" H 12950 12350 50  0000 L CNN
-F 2 "Package_DIP:DIP-14_W7.62mm" H 12800 11800 50  0001 C CNN
+F 2 "Package_SO:SOIC-16_3.9x9.9mm_P1.27mm" H 12800 11800 50  0001 C CNN
 F 3 "" H 12800 12200 50  0001 C CNN
 	2    12800 12200
@@
 F 0 "U301" H 12750 15100 50  0000 C CNN
 F 1 "ST26C32" H 12950 15250 50  0000 L CNN
-F 2 "Package_DIP:DIP-14_W7.62mm" H 12800 14700 50  0001 C CNN
+F 2 "Package_SO:SOIC-16_3.9x9.9mm_P1.27mm" H 12800 14700 50  0001 C CNN
 F 3 "" H 12800 15100 50  0001 C CNN
 	4    12800 15100
@@
 Wire Wire Line
 	15750 12400 15750 11950
-$Comp
-L aa-shared:+5V_X #PWR0114
-U 1 1 5EAF0A32
-P 15750 11900
-F 0 "#PWR0114" H 15750 11750 50  0001 C CNN
-F 1 "+5V_X" H 15765 12073 50  0000 C CNN
-F 2 "" H 15750 11900 50  0001 C CNN
-F 3 "" H 15750 11900 50  0001 C CNN
-	1    15750 11900
-	1    0    0    -1
-$EndComp
 Wire Wire Line
 	15650 13200 15750 13200
@@
 	17400 13100 17700 13100
 $Comp
-L power:GND #PWR?
+L power:GND #PWR0113
 U 1 1 5F141AF0
 P 16400 5050
-F 0 "#PWR?" H 16400 4800 50  0001 C CNN
+F 0 "#PWR0113" H 16400 4800 50  0001 C CNN
 F 1 "GND" H 16405 4877 50  0000 C CNN
 F 2 "" H 16400 5050 50  0001 C CNN
@@
 $EndComp
 $Comp
-L power:GND #PWR?
+L power:GND #PWR0130
 U 1 1 5F142A85
 P 16800 11600
-F 0 "#PWR?" H 16800 11350 50  0001 C CNN
+F 0 "#PWR0130" H 16800 11350 50  0001 C CNN
 F 1 "GND" H 16805 11427 50  0000 C CNN
 F 2 "" H 16800 11600 50  0001 C CNN
@@
 	10850 4100 11100 4100
 $Comp
-L aa-shared:GND_S #PWR?
+L aa-shared:GND_S #PWR0131
 U 1 1 5F20AE7C
 P 10900 7050
-F 0 "#PWR?" H 10900 6800 50  0001 C CNN
+F 0 "#PWR0131" H 10900 6800 50  0001 C CNN
 F 1 "GND_S" H 10905 6877 50  0000 C CNN
 F 2 "" H 10900 7050 50  0001 C CNN
@@
 	10900 7000 10900 7050
 $Comp
-L Connector:TestPoint TP?
+L Connector:TestPoint TP271
 U 1 1 5F20AE83
 P 10650 6900
-F 0 "TP?" H 10650 7100 50  0000 C BNN
+F 0 "TP271" H 10650 7100 50  0000 C BNN
 F 1 "TestPoint" V 10695 7088 50  0001 L CNN
 F 2 "aa-shared:TestPoint_Loop_D1.80mm_Drill1.0mm_Beaded" H 10850 6900 50  0001 C CNN
@@
 Connection ~ 11100 7000
 $Comp
-L aa-shared:GND_S #PWR?
+L aa-shared:GND_S #PWR0142
 U 1 1 5F52C7EE
 P 11250 13600
-F 0 "#PWR?" H 11250 13350 50  0001 C CNN
+F 0 "#PWR0142" H 11250 13350 50  0001 C CNN
 F 1 "GND_S" H 11255 13427 50  0000 C CNN
 F 2 "" H 11250 13600 50  0001 C CNN
@@
 	11250 13550 11500 13550
 $Comp
-L aa-shared:GND_S #PWR?
+L aa-shared:GND_S #PWR0143
 U 1 1 5F57CF82
 P 11250 10700
-F 0 "#PWR?" H 11250 10450 50  0001 C CNN
+F 0 "#PWR0143" H 11250 10450 50  0001 C CNN
 F 1 "GND_S" H 11255 10527 50  0000 C CNN
 F 2 "" H 11250 10700 50  0001 C CNN
@@
 	11250 10650 11500 10650
 Connection ~ 11500 10650
+Wire Wire Line
+	11850 1950 12150 1950
+$Comp
+L aa-shared:+5V_Y #PWR0114
+U 1 1 5F726085
+P 15750 11900
+F 0 "#PWR0114" H 15750 11750 50  0001 C CNN
+F 1 "+5V_Y" H 15765 12073 50  0000 C CNN
+F 2 "" H 15750 11900 50  0001 C CNN
+F 3 "" H 15750 11900 50  0001 C CNN
+	1    15750 11900
+	1    0    0    -1
+$EndComp
 $EndSCHEMATC
