File: hardware/aa-input-controller/aa-input-controller.sch (KiCad schematic (older format))
At the start: 26 parts, among them CN1 Barrel_Jack, CN2 Conn_01x02, CN3 Conn_01x03, CN4 Conn_01x03, CN5 6P6C, U2 NIS5132xx

Commit message: Update to use a shared schematic component/footprint library
Parts:
- CN5: footprint aa-input-controller:6P6C_Assmann_A-2014-1-4 -> aa-shared:6P6C_Assmann_A-2014-1-4
- D3: footprint aa-input-controller:D_SOD-923 -> aa-shared:D_SOD-923
- D6: symbol aa-input-controller:D5V0P4UR6SO -> aa-shared:D5V0P4UR6SO
- F1: footprint aa-input-controller:Fuseholder_Clip_5x20_Bel_FC-211-22 -> aa-shared:Fuseholder_Clip_5x20_Bel_FC-211-22
- U2: symbol aa-input-controller:NIS5132xx -> aa-shared:NIS5132xx
Changed lines of the file:
@@
 F 0 "F1" V 4303 2700 50  0000 C CNN
 F 1 "500mA" V 4394 2700 50  0000 C CNN
-F 2 "aa-input-controller:Fuseholder_Clip_5x20_Bel_FC-211-22" V 4430 2700 50  0001 C CNN
+F 2 "aa-shared:Fuseholder_Clip_5x20_Bel_FC-211-22" V 4430 2700 50  0001 C CNN
 F 3 "~" H 4500 2700 50  0001 C CNN
 	1    4500 2700
@@
 F 0 "D3" V 4954 3029 50  0000 L CNN
 F 1 "DF2S16FS" V 5045 3029 50  0000 L CNN
-F 2 "aa-input-controller:D_SOD-923" H 5000 2950 50  0001 C CNN
+F 2 "aa-shared:D_SOD-923" H 5000 2950 50  0001 C CNN
 F 3 "~" H 5000 2950 50  0001 C CNN
 	1    5000 2950
@@
 	5600 7200 5600 7600
 $Comp
-L aa-input-controller:+3V #PWR010
+L aa-shared:+3V #PWR010
 U 1 1 62386747
 P 4550 7100
@@
 	4100 2900 4100 2700
 $Comp
-L aa-input-controller:NIS5132xx U2
+L aa-shared:NIS5132xx U2
 U 1 1 5CEA4699
 P 5300 4450
@@
 $EndComp
 $Comp
-L aa-input-controller:D5V0P4UR6SO D6
+L aa-shared:D5V0P4UR6SO D6
 U 1 1 5EADDF25
 P 5100 7200
@@
 F 0 "CN5" H 6120 7154 50  0000 R CNN
 F 1 "6P6C" H 6120 7245 50  0000 R CNN
-F 2 "aa-input-controller:6P6C_Assmann_A-2014-1-4" V 6450 7175 50  0001 C CNN
+F 2 "aa-shared:6P6C_Assmann_A-2014-1-4" V 6450 7175 50  0001 C CNN
 F 3 "~" V 6450 7175 50  0001 C CNN
 	1    6450 7150

Commit message: Second run of PCBs for Amanita Arcade
Parts:
- removed C2: 1u, Capacitor_SMD:C_0805_2012Metric, symbol Device:C
- removed CN1: Barrel_Jack, Connector_BarrelJack:BarrelJack_Horizontal, symbol Connector:Barrel_Jack_Switch
- removed CN2: Conn_01x02, Connector_Wire:SolderWirePad_1x02_P7.62mm_Drill2.5mm, symbol Connector_Generic:Conn_01x02
- removed CN3, CN4: Conn_01x03, Connector_PinHeader_2.54mm:PinHeader_1x03_P2.54mm_Vertical, symbol Connector_Generic:Conn_01x03
- removed CN5: 6P6C, aa-shared:6P6C_Assmann_A-2014-1-4, symbol Connector:6P6C
- removed D3: DF2S16FS, aa-shared:D_SOD-923, symbol Device:D_Zener
- removed D6: D5V0P4UR6SO, Package_TO_SOT_SMD:SOT-23-6, symbol aa-shared:D5V0P4UR6SO
- removed F1: 500mA, aa-shared:Fuseholder_Clip_5x20_Bel_FC-211-22, symbol Device:Fuse
- removed JP5: SolderJumper_2_Open, Jumper:SolderJumper-2_P1.3mm_Open_RoundedPad1.0x1.5mm, symbol Jumper:SolderJumper_2_Open
- removed R15: 33, Resistor_SMD:R_0603_1608Metric, symbol Device:R
- removed R3, R4: 120, Resistor_SMD:R_0603_1608Metric, symbol Device:R
- removed R56: 10k, Resistor_SMD:R_0603_1608Metric, symbol Device:R
- removed R6, R7: 1k, Resistor_SMD:R_0603_1608Metric, symbol Device:R
- removed TP18, TP28, TP29, TP30, TP31: TestPoint, TestPoint:TestPoint_THTPad_D1.0mm_Drill0.5mm, symbol Connector:TestPoint
- removed U2: NIS5132xx, Package_DFN_QFN:DFN-10-1EP_3x3mm_P0.5mm_EP1.75x2.7mm, symbol aa-shared:NIS5132xx
- added A201: STM32F103_Bluepill, Module:Maple_Mini, symbol aa-shared:STM32F103_Bluepill
- added C101: 10u, Capacitor_THT:CP_Radial_D10.0mm_P2.50mm_P5.00mm, symbol Device:CP
- added C211, C221, C231, C241: 1u, Capacitor_SMD:C_0805_2012Metric, symbol Device:C
- added CN101: Conn_01x02, Connector_Wire:SolderWirePad_1x02_P5.08mm_Drill1.5mm, symbol Connector_Generic:Conn_01x02
- added CN201: INPUT, aa-shared:6P6C_Assmann_A-2014-1-4, symbol Connector:6P6C
- added CN202: Connector_Sony_Playstation_DualShock_Female, aa-shared:Connector_SonyPS2DualShock_Female, symbol aa-shared:Connector_Sony_Playstation_DualShock_Female
- added CN203, CN251: Conn_01x06_Male, Connector_PinHeader_2.54mm:PinHeader_1x06_P2.54mm_Vertical, symbol Connector:Conn_01x06_Male
- added CN211: BTN_R, aa-shared:6P6C_Assmann_A-2014-1-4, symbol Connector:6P6C
- added CN221: BTN_G, aa-shared:6P6C_Assmann_A-2014-1-4, symbol Connector:6P6C
- added CN231: BTN_B, aa-shared:6P6C_Assmann_A-2014-1-4, symbol Connector:6P6C
- added CN241: BTN_P, aa-shared:6P6C_Assmann_A-2014-1-4, symbol Connector:6P6C
- added FD1, FD2: Fiducial, Fiducial:Fiducial_1mm_Dia_2.54mm_Outer_CopperTop, symbol aa-shared:Fiducial
- added FD5, FD6: Fiducial, aa-shared:StencilAlignment_1.27mm, symbol aa-shared:Fiducial
- added Q211, Q221, Q231, Q241: MCH3484, Package_TO_SOT_SMD:SOT-323_SC-70, symbol Device:Q_NMOS_GSD
- added R201, R208: 1k, Resistor_SMD:R_0603_1608Metric, symbol Device:R
- added R202, R209: 120, Resistor_SMD:R_0603_1608Metric, symbol Device:R
- added R203, R204, R205, R206, R207, R211, R221, R231, R241: 4.7k, Resistor_SMD:R_0603_1608Metric, symbol Device:R
- added TP101: +12V, aa-shared:TestPoint_Loop_D1.80mm_Drill1.0mm_Beaded, symbol Connector:TestPoint
- added TP102: +5V, aa-shared:TestPoint_Loop_D1.80mm_Drill1.0mm_Beaded, symbol Connector:TestPoint
- added TP151, TP152, TP251, TP252, TP253, TP254, TP261, TP271, TP281, TP291: GND, aa-shared:TestPoint_Loop_D1.80mm_Drill1.0mm_Beaded, symbol Connector:TestPoint
- added TP211: BTN_R, aa-shared:TestPoint_Loop_D1.80mm_Drill1.0mm_Beaded, symbol Connector:TestPoint
- added TP212: PWM_R, aa-shared:TestPoint_Loop_D1.80mm_Drill1.0mm_Beaded, symbol Connector:TestPoint
- added TP213: LED_R, aa-shared:TestPoint_Loop_D1.80mm_Drill1.0mm_Beaded, symbol Connector:TestPoint
- added TP221: BTN_G, aa-shared:TestPoint_Loop_D1.80mm_Drill1.0mm_Beaded, symbol Connector:TestPoint
- added TP222: PWM_G, aa-shared:TestPoint_Loop_D1.80mm_Drill1.0mm_Beaded, symbol Connector:TestPoint
- added TP223: LED_G, aa-shared:TestPoint_Loop_D1.80mm_Drill1.0mm_Beaded, symbol Connector:TestPoint
- added TP231: BTN_B, aa-shared:TestPoint_Loop_D1.80mm_Drill1.0mm_Beaded, symbol Connector:TestPoint
- added TP232: PWM_B, aa-shared:TestPoint_Loop_D1.80mm_Drill1.0mm_Beaded, symbol Connector:TestPoint
- added TP233: LED_B, aa-shared:TestPoint_Loop_D1.80mm_Drill1.0mm_Beaded, symbol Connector:TestPoint
- added TP241: BTN_P, aa-shared:TestPoint_Loop_D1.80mm_Drill1.0mm_Beaded, symbol Connector:TestPoint
- added TP242: PWM_P, aa-shared:TestPoint_Loop_D1.80mm_Drill1.0mm_Beaded, symbol Connector:TestPoint
- added TP243: LED_P, aa-shared:TestPoint_Loop_D1.80mm_Drill1.0mm_Beaded, symbol Connector:TestPoint
- added U101: LM7805_TO220, Package_TO_SOT_THT:TO-220-3_Horizontal_TabDown, symbol Regulator_Linear:LM7805_TO220
- H1, H2, H3, H4: footprint MountingHole:MountingHole_4.3mm_M4_Pad_Via -> MountingHole:MountingHole_2.7mm_M2.5_Pad_Via
Connections:
- net labels added: +12V, +5V, BTN_B, BTN_G, BTN_P, BTN_R, LED_DRIVE_B, LED_DRIVE_G, LED_DRIVE_P, LED_DRIVE_R, PS2_ACK, PS2_ATT, PS2_CLK, PS2_CMD, PS2_DATA, PWM_B, PWM_G, PWM_P, PWM_R
- net labels removed: +3V, RX_DEBUG_S, RX_INPUT_S, TX_DEBUG_S, TX_INPUT_S, VDD
- wire segments 105 -> 246
- no-connect marks 2 -> 26
Other:
- moved on the sheet: H1, H2, H3, H4

Commit message: Minor board updates to fix issues discovered during build
Parts:
- R211, R221, R231, R241: value 4.7k -> 1k
Connections:
- net +5V: now also A201.38 (Pin_38); no longer A201.40 (Pin_40)
- no-connect marks 26 -> 27
Changed lines of the file:
@@
 Wire Wire Line
 	11150 7850 11150 7900
-Wire Wire Line
-	10700 7750 10800 7750
-Wire Wire Line
-	10800 7750 10800 7650
 NoConn ~ 9100 7750
 NoConn ~ 9100 7850
@@
 Wire Wire Line
 	9000 9650 9000 9750
-NoConn ~ 10700 7950
 NoConn ~ 9100 9350
 NoConn ~ 9100 7950
@@
 P 14400 10250
 F 0 "R211" H 14470 10296 50  0000 L CNN
-F 1 "4.7k" H 14470 10205 50  0000 L CNN
+F 1 "1k" H 14470 10205 50  0000 L CNN
 F 2 "Resistor_SMD:R_0603_1608Metric" V 14330 10250 50  0001 C CNN
 F 3 "~" H 14400 10250 50  0001 C CNN
@@
 P 14400 8700
 F 0 "R221" H 14470 8746 50  0000 L CNN
-F 1 "4.7k" H 14470 8655 50  0000 L CNN
+F 1 "1k" H 14470 8655 50  0000 L CNN
 F 2 "Resistor_SMD:R_0603_1608Metric" V 14330 8700 50  0001 C CNN
 F 3 "~" H 14400 8700 50  0001 C CNN
@@
 P 14400 7150
 F 0 "R231" H 14470 7196 50  0000 L CNN
-F 1 "4.7k" H 14470 7105 50  0000 L CNN
+F 1 "1k" H 14470 7105 50  0000 L CNN
 F 2 "Resistor_SMD:R_0603_1608Metric" V 14330 7150 50  0001 C CNN
 F 3 "~" H 14400 7150 50  0001 C CNN
@@
 P 14400 5600
 F 0 "R241" H 14470 5646 50  0000 L CNN
-F 1 "4.7k" H 14470 5555 50  0000 L CNN
+F 1 "1k" H 14470 5555 50  0000 L CNN
 F 2 "Resistor_SMD:R_0603_1608Metric" V 14330 5600 50  0001 C CNN
 F 3 "~" H 14400 5600 50  0001 C CNN
@@
 Wire Wire Line
 	12850 10450 12850 10500
+Wire Wire Line
+	10800 7950 10700 7950
+Wire Wire Line
+	10800 7650 10800 7950
+NoConn ~ 10700 7750
+NoConn ~ 8300 11700
 $EndSCHEMATC
