File: hardware/aa-stalk-receiver-lvds/aa-stalk-receiver-lvds.kicad_pcb (KiCad board)
At the start: 2 copper layers, 95.4 x 54 mm, 65 parts, among them CN101 Conn_01x02, CN102 6P6C, CN151 Conn_01x04, CN301 Conn_01x03, CN302 Conn_01x03, CN303 Conn_01x03, CN311 Conn_01x02, CN312 Conn_01x02, CN313 Conn_01x02, CN314 Conn_01x02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

Commit message: Fix silkscreen for stalk connectors
Other:
- board text added: "CN"
- board text added: "CP"
- board text added: "SN"
- board text added: "SP"
- board text removed: "PWM_CAP_N"
- board text removed: "PWM_CAP_P"
- board text removed: "RX_STALK_N"
- board text removed: "RX_STALK_P"
Changed lines of the file:
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@@
     (effects (font (size 0.508 0.508) (thickness 0.0762)))
   )
-  (gr_text PWM_CAP_N (at 122.809 93.98) (layer B.SilkS)
+  (gr_text CN (at 121.158 93.98) (layer B.SilkS)
     (effects (font (size 0.508 0.508) (thickness 0.0762)) (justify mirror))
   )
-  (gr_text PWM_CAP_P (at 113.538 92.71) (layer B.SilkS)
+  (gr_text CP (at 115.189 92.71) (layer B.SilkS)
     (effects (font (size 0.508 0.508) (thickness 0.0762)) (justify mirror))
   )
-  (gr_text RX_STALK_N (at 122.809 91.44) (layer B.SilkS)
+  (gr_text SN (at 121.158 91.44) (layer B.SilkS)
     (effects (font (size 0.508 0.508) (thickness 0.0762)) (justify mirror))
   )
-  (gr_text RX_STALK_P (at 113.538 90.17) (layer B.SilkS)
+  (gr_text SP (at 115.189 90.17) (layer B.SilkS)
     (effects (font (size 0.508 0.508) (thickness 0.0762)) (justify mirror))
   )
